File: HARDWARE/EDA/KiCad/RS485/RS485.sch (KiCad schematic (older format))
At the start: 46 parts

Commit message: add connectors
Parts:
- added J?: Conn_01x04_Male, Connector_JST:JST_EH_B4B-EH-A_1x04_P2.50mm_Vertical, symbol Connector:Conn_01x04_Male
- added J?: Conn_01x05_Male, Connector_JST:JST_EH_B5B-EH-A_1x05_P2.50mm_Vertical, symbol Connector:Conn_01x05_Male
Connections:
- net +3V3: now also J?.4 (Pin_4), J?.4 (Pin_4)
- net +5V: now also J?.5 (Pin_5)
- net A+: now also J?.2 (Pin_2)
- net B-: now also J?.3 (Pin_3)
- net GND: now also U?.5 (GND), J?.1 (Pin_1)
- net UART_RX: now also J?.2 (Pin_2)
- net UART_TX: now also J?.3 (Pin_3)
Other:
- moved on the sheet: D?, F?
Changed lines of the file:
@@
 L power:VSS #PWR?
 U 1 1 61BA5394
-P 4200 2250
-F 0 "#PWR?" H 4200 2100 50  0001 C CNN
-F 1 "VSS" H 4218 2423 50  0000 C CNN
-F 2 "" H 4200 2250 50  0001 C CNN
-F 3 "" H 4200 2250 50  0001 C CNN
-	1    4200 2250
-	-1   0    0    1
-$EndComp
-Wire Wire Line
-	4200 2250 4200 2150
+P 4200 2400
+F 0 "#PWR?" H 4200 2250 50  0001 C CNN
+F 1 "VSS" H 4218 2573 50  0000 C CNN
+F 2 "" H 4200 2400 50  0001 C CNN
+F 3 "" H 4200 2400 50  0001 C CNN
+	1    4200 2400
+	-1   0    0    1
+$EndComp
+Wire Wire Line
+	4200 2400 4200 2300
 $Comp
 L Device:R R?
@@
 Wire Wire Line
 	1850 3000 1700 3000
-Text GLabel 3600 1250 0    50   3State ~ 0
+Text GLabel 3600 1400 0    50   3State ~ 0
 B
-Text GLabel 3600 1750 0    50   3State ~ 0
+Text GLabel 3600 1900 0    50   3State ~ 0
 A
 $Comp
 L Device:D_TVS_ALT D?
 U 1 1 61FF4638
-P 4200 1500
-F 0 "D?" V 4154 1579 50  0000 L CNN
-F 1 "D_TVS_ALT" V 4245 1579 50  0000 L CNN
-F 2 "" H 4200 1500 50  0001 C CNN
-F 3 "~" H 4200 1500 50  0001 C CNN
-	1    4200 1500
+P 4200 1650
+F 0 "D?" V 4154 1729 50  0000 L CNN
+F 1 "D_TVS_ALT" V 4245 1729 50  0000 L CNN
+F 2 "" H 4200 1650 50  0001 C CNN
+F 3 "~" H 4200 1650 50  0001 C CNN
+	1    4200 1650
 	0    -1   1    0
 $EndComp
 Wire Wire Line
-	4200 1750 4200 1650
-Wire Wire Line
-	4200 1750 3600 1750
-Wire Wire Line
-	4200 1250 4200 1350
-Wire Wire Line
-	4200 1250 3600 1250
+	4200 1900 4200 1800
+Wire Wire Line
+	4200 1900 3600 1900
+Wire Wire Line
+	4200 1400 4200 1500
+Wire Wire Line
+	4200 1400 3600 1400
 $Comp
 L Device:D_TVS_ALT D?
 U 1 1 6200DF80
-P 4200 1000
-F 0 "D?" V 4154 1079 50  0000 L CNN
-F 1 "D_TVS_ALT" V 4245 1079 50  0000 L CNN
-F 2 "" H 4200 1000 50  0001 C CNN
-F 3 "~" H 4200 1000 50  0001 C CNN
-	1    4200 1000
+P 4200 1150
+F 0 "D?" V 4154 1229 50  0000 L CNN
+F 1 "D_TVS_ALT" V 4245 1229 50  0000 L CNN
+F 2 "" H 4200 1150 50  0001 C CNN
+F 3 "~" H 4200 1150 50  0001 C CNN
+	1    4200 1150
 	0    -1   1    0
 $EndComp
 Wire Wire Line
-	4200 1150 4200 1250
-Connection ~ 4200 1250
+	4200 1300 4200 1400
+Connection ~ 4200 1400
 $Comp
 L Device:D_TVS_ALT D?
 U 1 1 620125B3
-P 4200 2000
-F 0 "D?" V 4154 2079 50  0000 L CNN
-F 1 "D_TVS_ALT" V 4245 2079 50  0000 L CNN
-F 2 "" H 4200 2000 50  0001 C CNN
-F 3 "~" H 4200 2000 50  0001 C CNN
-	1    4200 2000
+P 4200 2150
+F 0 "D?" V 4154 2229 50  0000 L CNN
+F 1 "D_TVS_ALT" V 4245 2229 50  0000 L CNN
+F 2 "" H 4200 2150 50  0001 C CNN
+F 3 "~" H 4200 2150 50  0001 C CNN
+	1    4200 2150
 	0    -1   1    0
 $EndComp
 Wire Wire Line
-	4200 1850 4200 1750
-Connection ~ 4200 1750
+	4200 2000 4200 1900
+Connection ~ 4200 1900
 $Comp
 L power:VCC #PWR?
 U 1 1 6201B2B7
-P 4200 750
-F 0 "#PWR?" H 4200 600 50  0001 C CNN
-F 1 "VCC" H 4217 923 50  0000 C CNN
-F 2 "" H 4200 750 50  0001 C CNN
-F 3 "" H 4200 750 50  0001 C CNN
-	1    4200 750
-	1    0    0    -1
-$EndComp
-Wire Wire Line
-	4200 750  4200 850
+P 4200 900
+F 0 "#PWR?" H 4200 750 50  0001 C CNN
+F 1 "VCC" H 4217 1073 50  0000 C CNN
+F 2 "" H 4200 900 50  0001 C CNN
+F 3 "" H 4200 900 50  0001 C CNN
+	1    4200 900
+	1    0    0    -1
+$EndComp
+Wire Wire Line
+	4200 900  4200 1000
 $Comp
 L Device:Polyfuse F?
 U 1 1 6204742C
-P 4550 1250
-F 0 "F?" V 4325 1250 50  0000 C CNN
-F 1 "Polyfuse" V 4416 1250 50  0000 C CNN
-F 2 "" H 4600 1050 50  0001 L CNN
-F 3 "~" H 4550 1250 50  0001 C CNN
-	1    4550 1250
+P 4550 1400
+F 0 "F?" V 4325 1400 50  0000 C CNN
+F 1 "Polyfuse" V 4416 1400 50  0000 C CNN
+F 2 "" H 4600 1200 50  0001 L CNN
+F 3 "~" H 4550 1400 50  0001 C CNN
+	1    4550 1400
 	0    1    1    0
 $EndComp
 Wire Wire Line
-	4400 1250 4200 1250
+	4400 1400 4200 1400
 $Comp
 L Device:Polyfuse F?
 U 1 1 6204D72D
-P 4550 1750
-F 0 "F?" V 4325 1750 50  0000 C CNN
-F 1 "Polyfuse" V 4416 1750 50  0000 C CNN
-F 2 "" H 4600 1550 50  0001 L CNN
-F 3 "~" H 4550 1750 50  0001 C CNN
-	1    4550 1750
+P 4550 1900
+F 0 "F?" V 4325 1900 50  0000 C CNN
+F 1 "Polyfuse" V 4416 1900 50  0000 C CNN
+F 2 "" H 4600 1700 50  0001 L CNN
+F 3 "~" H 4550 1900 50  0001 C CNN
+	1    4550 1900
 	0    1    1    0
 $EndComp
 Wire Wire Line
-	4400 1750 4200 1750
-Text GLabel 4800 1250 2    50   3State ~ 0
+	4400 1900 4200 1900
+Text GLabel 4800 1400 2    50   3State ~ 0
 B-
 Wire Wire Line
-	4800 1250 4700 1250
-Text GLabel 4800 1750 2    50   3State ~ 0
+	4800 1400 4700 1400
+Text GLabel 4800 1900 2    50   3State ~ 0
 A+
 Wire Wire Line
-	4800 1750 4700 1750
+	4800 1900 4700 1900
+Wire Wire Line
+	6950 3950 6950 4050
+$Comp
+L power:VSS #PWR?
+U 1 1 61BC455F
+P 6950 4050
+F 0 "#PWR?" H 6950 3900 50  0001 C CNN
+F 1 "VSS" H 6968 4223 50  0000 C CNN
+F 2 "" H 6950 4050 50  0001 C CNN
+F 3 "" H 6950 4050 50  0001 C CNN
+	1    6950 4050
+	-1   0    0    1
+$EndComp
+$Comp
+L Connector:Conn_01x04_Male J?
+U 1 1 61BD7C0A
+P 8250 1550
+F 0 "J?" H 8222 1432 50  0000 R CNN
+F 1 "Conn_01x04_Male" H 8222 1523 50  0000 R CNN
+F 2 "Connector_JST:JST_EH_B4B-EH-A_1x04_P2.50mm_Vertical" H 8250 1550 50  0001 C CNN
+F 3 "~" H 8250 1550 50  0001 C CNN
+	1    8250 1550
+	-1   0    0    1
+$EndComp
+Text GLabel 7950 1450 0    50   3State ~ 0
+B-
+Text GLabel 7950 1550 0    50   3State ~ 0
+A+
+Wire Wire Line
+	6400 1700 6400 1800
+$Comp
+L power:VSS #PWR?
+U 1 1 61BF7B9E
+P 6400 1800
+F 0 "#PWR?" H 6400 1650 50  0001 C CNN
+F 1 "VSS" H 6418 1973 50  0000 C CNN
+F 2 "" H 6400 1800 50  0001 C CNN
+F 3 "" H 6400 1800 50  0001 C CNN
+	1    6400 1800
+	-1   0    0    1
+$EndComp
+Wire Wire Line
+	6400 1700 6500 1700
+Wire Wire Line
+	7950 1550 8050 1550
+Wire Wire Line
+	7950 1450 8050 1450
+$Comp
+L power:VCC #PWR?
+U 1 1 61C11188
+P 7950 1250
+F 0 "#PWR?" H 7950 1100 50  0001 C CNN
+F 1 "VCC" H 7967 1423 50  0000 C CNN
+F 2 "" H 7950 1250 50  0001 C CNN
+F 3 "" H 7950 1250 50  0001 C CNN
+	1    7950 1250
+	1    0    0    -1
+$EndComp
+Wire Wire Line
+	7950 1250 7950 1350
+Wire Wire Line
+	7950 1350 8050 1350
+$Comp
+L Connector:Conn_01x05_Male J?
+U 1 1 61C1D525
+P 6700 1500
+F 0 "J?" H 6672 1432 50  0000 R CNN
+F 1 "Conn_01x05_Male" H 6672 1523 50  0000 R CNN
+F 2 "Connector_JST:JST_EH_B5B-EH-A_1x05_P2.50mm_Vertical" H 6700 1500 50  0001 C CNN
+F 3 "~" H 6700 1500 50  0001 C CNN
+	1    6700 1500
+	-1   0    0    1
+$EndComp
+Text GLabel 6350 1500 0    50   Input ~ 0
+UART_TX
+Text GLabel 6350 1600 0    50   Output ~ 0
+UART_RX
+Wire Wire Line
+	6350 1600 6500 1600
+Wire Wire Line
+	6350 1500 6500 1500
+$Comp
+L power:+5V #PWR?
+U 1 1 61C7D8E0
+P 6400 1200
+F 0 "#PWR?" H 6400 1050 50  0001 C CNN
+F 1 "+5V" H 6415 1373 50  0000 C CNN
+F 2 "" H 6400 1200 50  0001 C CNN
+F 3 "" H 6400 1200 50  0001 C CNN
+	1    6400 1200
+	1    0    0    -1
+$EndComp
+Wire Wire Line
+	6400 1200 6400 1300
+Wire Wire Line
+	6400 1300 6500 1300
+$Comp
+L power:VCC #PWR?
+U 1 1 61C93CEC
+P 6200 1200
+F 0 "#PWR?" H 6200 1050 50  0001 C CNN
+F 1 "VCC" H 6217 1373 50  0000 C CNN
+F 2 "" H 6200 1200 50  0001 C CNN
+F 3 "" H 6200 1200 50  0001 C CNN
+	1    6200 1200
+	1    0    0    -1
+$EndComp
+Wire Wire Line
+	6200 1200 6200 1400
+Wire Wire Line
+	6200 1400 6500 1400
 $EndSCHEMATC

Commit message: schematic revised
Parts:
- removed D? (x3): D_TVS_ALT, symbol Device:D_TVS_ALT
- added D1, D2, D3: TVS 15.3V, Diode_THT:D_DO-201AE_P15.24mm_Horizontal, symbol Diode:1N62xxCA
- F1, F2: renamed from F?; footprint (none) -> Fuse:Fuse_Bourns_MF-RG300
- U1: renamed from U?; footprint (none) -> Package_DIP:DIP-14_W7.62mm_LongPads
- gave numbers to parts that had none: 36
Connections:
- net +3V3: now also D1.1 (A1)
- net A: now also D2.2 (A2), D3.1 (A1)
- net B: now also D1.2 (A2), D2.1 (A1)
- net GND: now also D3.2 (A2)
